File: squirrelbrain.kicad_pcb (KiCad board)
At the start: 2 copper layers, 27 x 27 mm, 32 parts, among them J1 BM02B-SRSS-TB_LF__SN_, J2 Conn_01x03, J3 BM02B-SRSS-TB_LF__SN_, J4 BATT, J5 BLDC_PWR, J6 GPIO1, U1 RPM5.0-6.0, U2 TPS1HB08BQPWPRQ1, U3 TPS22992SRXNR, U4 SEEEDUINO-XIAO-ESP32S3, U5 THVD1420DRLR, U6 SN74LVC2G125DCUR, U7 THVD1420DRLR

Commit message: generate gerbers
Parts:
- removed R4: 10k, Resistor_SMD:R_0402_1005Metric
- added G***: LOGO, LOGO, F.Cu at (62.8, 47.9)
- added G***: LOGO, LOGO, B.Cu at (59.1, 39.7)
- added G***: LOGO, LOGO, B.Cu at (59.0, 37.9)
- added G***: LOGO, LOGO, B.Cu at (40.7, 50.3)
- added R9: 1k, Resistor_SMD:R_0402_1005Metric, B.Cu at (56.6, 37.7)
- added TP1: TestPoint, squirrelbrain:TestPoint_Pad_Rect, B.Cu at (58.4, 37.7)
- added TP6: TestPoint, squirrelbrain:TestPoint_Pad_Rect, B.Cu at (58.4, 40.1)
- R1: value 1k -> 390R
- moved R8 0.95 mm to (55.6, 37.7), turned to 90 degrees
- moved C4 0.64 mm to (60.6, 55.9)
- moved G*** 0.52 mm to (60.9, 55.6)
- moved R6 0.15 mm to (56.5, 40.2), turned to 0 degrees
- moved U3 0.14 mm to (56.8, 42.2)
- moved D1 0.08 mm to (56.5, 39.2)
Connections:
- U4 pad 1: /MOTOR_ON -> Net-(U4-PA02_A0_D0)
Routing:
- net GND: track 15.6 -> 38.1 mm, vias 34 -> 44
- net Net-(U4-PA02_A0_D0): track 0.00 -> 18.2 mm, vias 0 -> 1
- net /MOTOR_ON: track 38.3 -> 26.6 mm
- net /UART2_DE: track 18.2 -> 29.2 mm
- net /RS485_0A: track 7.84 -> 12.3 mm, vias 2 -> 0
- net Net-(J6-Pin_1): track 23.2 -> 20.9 mm
- net /SNS: track 19.3 -> 18.1 mm
- net Net-(U2-ILIM): track 5.23 -> 5.88 mm
- net Net-(J5-Pin_2): track 9.10 -> 9.31 mm, vias 5 -> 4
Other:
- board text added: "3V3 RS485"
- board text removed: "G"
- board text removed: "JST-EH"
- board text removed: "RS485"

Commit message: add schematic labels just for reference
Connections:
- net Net-(D1-K) renamed /5V_ESP
- net Net-(J5-Pin_2) renamed /BLDC_PWR
- net Net-(J6-Pin_1) renamed /SNS_IO
- net Net-(U4-PA02_A0_D0) renamed /MOTOR_ON_IO
